Commit message: mid term project init

File: urdf/sawyer/sawyer.urdf (robot description, URDF)
Before this commit: robot sawyer, 24 links, 23 joints
Links:
- link sawyer_head: geometry collision sphere radius=0.18; visual mesh filename=meshes/sawyer_pv/head.stl
- link sawyer_link_0: geometry collision sphere radius=0.07; visual mesh filename=meshes/sawyer_mp3/l0.stl
- link sawyer_link_1: geometry collision sphere radius=0.07; visual mesh filename=meshes/sawyer_mp3/l1.stl
- link sawyer_link_2: geometry collision cylinder length=0.34 radius=0.06; visual mesh filename=meshes/sawyer_pv/l2.stl
- link sawyer_link_3: geometry collision sphere radius=0.06; visual mesh filename=meshes/sawyer_pv/l3.stl
- link sawyer_link_4: geometry collision cylinder length=0.30 radius=0.045; visual mesh filename=meshes/sawyer_pv/l4.stl
- link sawyer_link_5: geometry collision sphere radius=0.06; visual mesh filename=meshes/sawyer_pv/l5.stl
- link sawyer_link_6: geometry collision cylinder length=0.05 radius=0.055; visual mesh filename=meshes/sawyer_mp1/l6.stl
- link sawyer_pedestal: geometry collision cylinder length=0.62 radius=0.18; visual mesh filename=meshes/sawyer_pv/pedestal.stl
- link sawyer_right_arm_base_link: geometry collision cylinder length=0.24 radius=0.08; visual mesh filename=meshes/sawyer_pv/base.stl
