Commit message: practice 4 upload

File: urdf/doosan/doosan_with_robotiq140.urdf (robot description, URDF)
Before this commit: robot doosan, 24 links, 23 joints
Links:
- link doosan_pedestal: geometry collision cylinder length=0.62 radius=0.18; visual mesh filename=meshes/doosan_pedestal/pedestal.stl
